Commit message: zfshen,修改

File: src/ur_description/urdf/ur5_support.urdf (robot description, URDF)
Before this commit: robot ur5, 15 links, 14 joints
Links:
- removed link world_link
- added link arm_world_link
- added link base_support_cylinder_link_0; collision cylinder length=0.15 radius=0.12; visual cylinder length=0.15 radius=0.16
- added link table_leg_link_1; collision box size=0.06 0.03 0.725; visual box size=0.06 0.03 0.725
- added link table_leg_link_2; collision box size=0.06 0.03 0.725; visual box size=0.06 0.03 0.725
- added link table_leg_link_3; collision box size=0.06 0.03 0.725; visual box size=0.06 0.03 0.725
- added link table_leg_link_4; collision box size=0.06 0.03 0.725; visual box size=0.06 0.03 0.725
- added link table_top_link; collision box size=1.4 0.7 0.025; visual box size=1.4 0.7 0.025
- link base_support_box_link: geometry collision box size=0.1 0.40 0.1; visual box size=0.1 0.46 0.1
- link base_support_cylinder_link: geometry collision cylinder length=1.0 radius=0.05; visual cylinder length=1.0 radius=0.085
- link base_support_cylinder_link_2: geometry collision cylinder length=0.5 radius=0.05; visual cylinder length=0.5 radius=0.05
Joints:
- added joint cylinde_cylinder_link_0: type fixed, parent base_support_cylinder_link_0, child base_support_cylinder_link, origin xyz=0.0 0.0 0.575 rpy=0.0 0.0 0.0
- added joint table_leg_joint_1: type fixed, parent table_top_link, child table_leg_link_1, origin xyz=0.67 0.335 -0.3625 rpy=0.0 0.0 0.0
- added joint table_leg_joint_2: type fixed, parent table_top_link, child table_leg_link_2, origin xyz=0.67 -0.335 -0.3625 rpy=0.0 0.0 0.0
- added joint table_leg_joint_3: type fixed, parent table_top_link, child table_leg_link_3, origin xyz=-0.67 0.335 -0.3625 rpy=0.0 0.0 0.0
- added joint table_leg_joint_4: type fixed, parent table_top_link, child table_leg_link_4, origin xyz=-0.67 -0.335 -0.3625 rpy=0.0 0.0 0.0
- added joint table_top_joint: type fixed, parent world, child table_top_link, origin xyz=0.0 0.45 0.725 rpy=0.0 0.0 0.0
- joint base_support_joint_L: parent world_link -> arm_world_link
- joint base_world_joint: child world_link -> arm_world_link; origin xyz=0.0 0.25 0.0 rpy=0.0 0.0 -1.5708 -> xyz=0.0 0.23 0.0 rpy=0.0 0.0 -1.5708
- joint box_cylinder_link: origin xyz=0.0 0.0 0.25 rpy=0.0 0.0 0.0 -> xyz=0.0 0.0 0.3 rpy=0.0 0.0 0.0
- joint cylinde_cylinder_link: origin xyz=0.0 0.0 0.8 rpy=0.0 0.0 0.0 -> xyz=0.0 0.0 0.75 rpy=0.0 0.0 0.0
- joint world_joint: child base_support_cylinder_link -> base_support_cylinder_link_0; origin xyz=0.0 0.0 0.6 rpy=0.0 0.0 1.5708 -> xyz=0.0 0.0 0.075 rpy=0.0 0.0 1.5708
